File: KiCad/Amiga_DB23_video_adapter.sch (KiCad schematic (older format))
At the start: 17 parts, among them J1 DB23_Female, J2 Conn_02x06_Odd_Even, J3 Conn_01x03, SW1 SW_SPDT, U1 74HCT2G17, U2 74HCT2G14, X1 K50-HC0CSE28.6363MR

Commit message: Add new design based on a THS7374IPWR, 28M oscillator circuit, remove SolderJumper, complete re-design and re-route
Parts:
- removed J2: Conn_02x06_Odd_Even, Connector_PinHeader_2.00mm:PinHeader_2x06_P2.00mm_Vertical, symbol Connector_Generic:Conn_02x06_Odd_Even
- removed J3: Conn_01x03, Connector_PinHeader_2.00mm:PinHeader_1x03_P2.00mm_Vertical, symbol Connector_Generic:Conn_01x03
- removed JP1: SolderJumper_3_Open, Jumper:SolderJumper-3_P1.3mm_Open_Pad1.0x1.5mm_NumberLabels, symbol Jumper:SolderJumper_3_Open
- removed X1: K50-HC0CSE28.6363MR, Oscillator:Oscillator_SMD_SeikoEpson_SG8002CA-4Pin_7.0x5.0mm, symbol Oscillator:SG-8002CA
- added C5, C6: 32 pF, Capacitor_SMD:C_0603_1608Metric_Pad1.08x0.95mm_HandSolder, symbol Device:C_Small
- added C7: 0.1uF, Capacitor_SMD:C_0603_1608Metric_Pad1.08x0.95mm_HandSolder, symbol Device:C_Small
- added J2, J3: Conn_01x06, Connector_PinHeader_2.00mm:PinHeader_1x06_P2.00mm_Vertical, symbol Connector_Generic:Conn_01x06
- added J5, J6, J?: Conn_01x02, Connector_PinHeader_2.00mm:PinHeader_1x02_P2.00mm_Vertical, symbol Connector_Generic:Conn_01x02
- added R10: 1k, Resistor_SMD:R_0603_1608Metric_Pad0.98x0.95mm_HandSolder, symbol Device:R_Small
- added R11: 2.2M, Resistor_SMD:R_0603_1608Metric_Pad0.98x0.95mm_HandSolder, symbol Device:R_Small
- added R12: 150, Resistor_SMD:R_1206_3216Metric_Pad1.30x1.75mm_HandSolder, symbol Device:R_Small
- added R6, R7, R8: 75, Resistor_SMD:R_0603_1608Metric_Pad0.98x0.95mm_HandSolder, symbol Device:R_Small
- added R9: 100, Resistor_SMD:R_1206_3216Metric_Pad1.30x1.75mm_HandSolder, symbol Device:R_Small
- added RN1: R_Pack04, Amiga_DB23_video_adapter:RESCAF80P320X160X60-8N, symbol Device:R_Pack04
- added U3: THS7374IPWR, Package_SO:TSSOP-14_4.4x5mm_P0.65mm, symbol Amiga_DB23_video_adapter:THS7374IPWR
- added U4: 74LVC1GX04, Package_SO:TSOP-6_1.65x3.05mm_P0.95mm, symbol Amiga_DB23_video_adapter:74LVC1GX04
- added Y1: CL=16pF, Crystal:Crystal_SMD_SeikoEpson_FA238-4Pin_3.2x2.5mm, symbol Device:Crystal_GND24
- C2, C4: footprint Capacitor_SMD:C_0805_2012Metric_Pad1.15x1.40mm_HandSolder -> Capacitor_SMD:C_0603_1608Metric_Pad1.08x0.95mm_HandSolder
- J1: symbol Connector:DB23_Female -> Amiga_DB23_video_adapter:DB23_Female-Connector
Connections:
- net labels added: AMIGA_B, AMIGA_G, AMIGA_R, B, G, R
- net labels removed: ToAgnusPin41
- wire segments 26 -> 56
- no-connect marks 10 -> 11
Other:
- moved on the sheet: C1

Commit message: Improve GND-stitching and fix silkscreen text and add new revision identifier
Parts:
- gave numbers to parts that had none: 1
Connections:
- net OE is gone; now on net XCLKEN: J6.1 (Pin_1), U2.6 (1Y)
- net XCLKEN: no longer J1.2, J6.2 (Pin_2), U2.1 (1A), U2.4 (2Y)
- new net XCLKEN_n: J1.2, J6.2 (Pin_2), U2.1 (1A), U2.4 (2Y)
Other:
- moved on the sheet: C4
Changed lines of the file:
@@
 $EndComp
 Text GLabel 4700 2750 3    50   Input ~ 0
-XCLKEN
+XCLKEN_n
 Text GLabel 3900 7050 3    50   Input ~ 0
 VCC
@@
 Connection ~ 1950 3900
 Text GLabel 3200 3900 2    50   Output ~ 0
-XCLKEN
-Text GLabel 3200 3500 2    50   Output ~ 0
-OE
+XCLKEN_n
 Text GLabel 2300 3700 0    50   Input ~ 0
 GND
-Text GLabel 3500 3700 2    50   Input ~ 0
+Text GLabel 3850 3700 2    50   Input ~ 0
 VCC
 $Comp
 L Device:C_Small C4
 U 1 1 604F7F40
-P 3500 3600
-F 0 "C4" H 3400 3600 50  0000 R CNN
-F 1 "0.1uF" H 3600 3600 50  0000 L CNN
-F 2 "Capacitor_SMD:C_0603_1608Metric_Pad1.08x0.95mm_HandSolder" H 3500 3600 50  0001 C CNN
-F 3 "~" H 3500 3600 50  0001 C CNN
-	1    3500 3600
-	1    0    0    -1
-$EndComp
-Text GLabel 3500 3500 2    50   Input ~ 0
-GND
-Wire Wire Line
-	3200 3700 3500 3700
+P 3850 3600
+F 0 "C4" H 3750 3600 50  0000 R CNN
+F 1 "0.1uF" H 3950 3600 50  0000 L CNN
+F 2 "Capacitor_SMD:C_0603_1608Metric_Pad1.08x0.95mm_HandSolder" H 3850 3600 50  0001 C CNN
+F 3 "~" H 3850 3600 50  0001 C CNN
+	1    3850 3600
+	1    0    0    -1
+$EndComp
+Text GLabel 3850 3500 2    50   Input ~ 0
+GND
 $Comp
 L Device:R R4
@@
 	1150 3900 1150 4050
 Text GLabel 2300 3500 0    50   Input ~ 0
-XCLKEN
+XCLKEN_n
 Text GLabel 2250 2750 0    50   Input ~ 0
 VCC
@@
 $EndComp
 Text GLabel 3250 4850 3    50   Input ~ 0
-XCLKEN
-Text GLabel 3150 4850 3    50   Input ~ 0
-OE
-$Comp
-L Connector_Generic:Conn_01x02 J?
+XCLKEN_n
+$Comp
+L Connector_Generic:Conn_01x02 J4
 U 1 1 6A423A43
 P 3650 4650
-F 0 "J?" V 3650 4800 50  0000 R CNN
+F 0 "J4" V 3650 4800 50  0000 R CNN
 F 1 "Conn_01x02" V 3750 4900 50  0000 R CNN
 F 2 "Connector_PinHeader_2.00mm:PinHeader_1x02_P2.00mm_Vertical" H 3650 4650 50  0001 C CNN
@@
 Text GLabel 3750 4850 3    50   Input ~ 0
 GND
+Wire Wire Line
+	3200 3700 3850 3700
+Text GLabel 3200 3500 2    50   Output ~ 0
+XCLKEN
+Text GLabel 3150 4850 3    50   Input ~ 0
+XCLKEN
 $EndSCHEMATC

Commit message: Swap references C2,C3. Swap references C5,C7. Swap references R1,R9. Swap references R4,R12
Parts:
- renumbered C3 to C2, C2 to C3, C7 to C5, C5 to C7, R9 to R1, R4 to R12, R12 to R4, R1 to R9
Changed lines of the file:
@@
 NoConn ~ 6200 2750
 $Comp
-L Device:R R1
+L Device:R R9
 U 1 1 5DD5FE14
 P 6300 3400
-F 0 "R1" H 6150 3400 50  0000 L CNN
+F 0 "R9" H 6150 3400 50  0000 L CNN
 F 1 "330" V 6300 3350 50  0000 L CNN
 F 2 "Resistor_SMD:R_0805_2012Metric_Pad1.15x1.40mm_HandSolder" V 6230 3400 50  0001 C CNN
@@
 GND
 $Comp
-L Device:C_Small C2
+L Device:C_Small C3
 U 1 1 604C0786
 P 7600 4400
-F 0 "C2" H 7500 4400 50  0000 R CNN
+F 0 "C3" H 7500 4400 50  0000 R CNN
 F 1 "0.1uF" H 7700 4400 50  0000 L CNN
 F 2 "Capacitor_SMD:C_0603_1608Metric_Pad1.08x0.95mm_HandSolder" H 7600 4400 50  0001 C CNN
@@
 GND
 $Comp
-L Device:C_Small C3
+L Device:C_Small C2
 U 1 1 604D1DD2
 P 1950 4000
-F 0 "C3" H 2050 4150 50  0000 R CNN
+F 0 "C2" H 2050 4150 50  0000 R CNN
 F 1 "0.1uF" H 2042 3955 50  0000 L CNN
 F 2 "Capacitor_SMD:C_0805_2012Metric_Pad1.15x1.40mm_HandSolder" H 1950 4000 50  0001 C CNN
@@
 GND
 $Comp
-L Device:R R4
+L Device:R R12
 U 1 1 6053876C
 P 1150 3600
-F 0 "R4" H 1200 3600 50  0000 L CNN
+F 0 "R12" H 1200 3600 50  0000 L CNN
 F 1 "10k" V 1150 3500 50  0000 L CNN
 F 2 "Resistor_SMD:R_0805_2012Metric_Pad1.15x1.40mm_HandSolder" V 1080 3600 50  0001 C CNN
@@
 	4750 3650 4750 3800
 $Comp
-L Device:R_Small R9
+L Device:R_Small R1
 U 1 1 6A27D6DD
 P 5000 3300
-F 0 "R9" H 5059 3346 50  0000 L CNN
+F 0 "R1" H 5059 3346 50  0000 L CNN
 F 1 "100" H 5059 3255 50  0000 L CNN
 F 2 "Resistor_SMD:R_1206_3216Metric_Pad1.30x1.75mm_HandSolder" H 5000 3300 50  0001 C CNN
@@
 	2300 6250 2200 6250
 $Comp
-L Device:C_Small C5
+L Device:C_Small C7
 U 1 1 6A2C1303
 P 2300 5950
-F 0 "C5" V 2150 5950 50  0000 C CNN
+F 0 "C7" V 2150 5950 50  0000 C CNN
 F 1 "32 pF" V 2050 6000 50  0000 C CNN
 F 2 "Capacitor_SMD:C_0603_1608Metric_Pad1.08x0.95mm_HandSolder" H 2300 5950 50  0001 C CNN
@@
 GND
 $Comp
-L Device:R_Small R12
+L Device:R_Small R4
 U 1 1 6A39DE05
 P 4500 6700
-F 0 "R12" V 4600 6650 50  0000 L CNN
+F 0 "R4" V 4600 6650 50  0000 L CNN
 F 1 "150" V 4400 6650 50  0000 L CNN
 F 2 "Resistor_SMD:R_1206_3216Metric_Pad1.30x1.75mm_HandSolder" H 4500 6700 50  0001 C CNN
@@
 	4600 6700 4850 6700
 $Comp
-L Device:C_Small C7
+L Device:C_Small C5
 U 1 1 6A3BE810
 P 3800 6900
-F 0 "C7" V 3700 6850 50  0000 R CNN
+F 0 "C5" V 3700 6850 50  0000 R CNN
 F 1 "0.1uF" V 3900 6750 50  0000 L CNN
 F 2 "Capacitor_SMD:C_0603_1608Metric_Pad1.08x0.95mm_HandSolder" H 3800 6900 50  0001 C CNN

Commit message: Swap references R5,R9. Swap references R10,R12
Parts:
- renumbered R12 to R10, R10 to R12, R9 to R5, R5 to R9
Changed lines of the file:
@@
 NoConn ~ 6200 2750
 $Comp
-L Device:R R9
+L Device:R R5
 U 1 1 5DD5FE14
 P 6300 3400
-F 0 "R9" H 6150 3400 50  0000 L CNN
+F 0 "R5" H 6150 3400 50  0000 L CNN
 F 1 "330" V 6300 3350 50  0000 L CNN
 F 2 "Resistor_SMD:R_0805_2012Metric_Pad1.15x1.40mm_HandSolder" V 6230 3400 50  0001 C CNN
@@
 GND
 $Comp
-L Device:R R12
+L Device:R R10
 U 1 1 6053876C
 P 1150 3600
-F 0 "R12" H 1200 3600 50  0000 L CNN
+F 0 "R10" H 1200 3600 50  0000 L CNN
 F 1 "10k" V 1150 3500 50  0000 L CNN
 F 2 "Resistor_SMD:R_0805_2012Metric_Pad1.15x1.40mm_HandSolder" V 1080 3600 50  0001 C CNN
@@
 $EndComp
 $Comp
-L Device:R R5
+L Device:R R9
 U 1 1 6053FB6E
 P 1500 3900
-F 0 "R5" V 1600 3850 50  0000 L CNN
+F 0 "R9" V 1600 3850 50  0000 L CNN
 F 1 "10k" V 1500 3850 50  0000 L CNN
 F 2 "Resistor_SMD:R_0805_2012Metric_Pad1.15x1.40mm_HandSolder" V 1430 3900 50  0001 C CNN
@@
 GND
 $Comp
-L Device:R_Small R10
+L Device:R_Small R12
 U 1 1 6A317F34
 P 2800 6550
-F 0 "R10" V 2700 6500 50  0000 L CNN
+F 0 "R12" V 2700 6500 50  0000 L CNN
 F 1 "1k" V 2800 6500 50  0000 L CNN
 F 2 "Resistor_SMD:R_0603_1608Metric_Pad0.98x0.95mm_HandSolder" H 2800 6550 50  0001 C CNN

Commit message: Swap references R11,R12 and fix positioning of R10
Parts:
- renumbered R12 to R11, R11 to R12
Changed lines of the file:
@@
 GND
 $Comp
-L Device:R_Small R12
+L Device:R_Small R11
 U 1 1 6A317F34
 P 2800 6550
-F 0 "R12" V 2700 6500 50  0000 L CNN
+F 0 "R11" V 2700 6500 50  0000 L CNN
 F 1 "1k" V 2800 6500 50  0000 L CNN
 F 2 "Resistor_SMD:R_0603_1608Metric_Pad0.98x0.95mm_HandSolder" H 2800 6550 50  0001 C CNN
@@
 Connection ~ 2500 6550
 $Comp
-L Device:R_Small R11
+L Device:R_Small R12
 U 1 1 6A31A283
 P 3150 6250
-F 0 "R11" H 2950 6200 50  0000 L CNN
+F 0 "R12" H 2950 6200 50  0000 L CNN
 F 1 "2.2M" H 2900 6300 50  0000 L CNN
 F 2 "Resistor_SMD:R_0603_1608Metric_Pad0.98x0.95mm_HandSolder" H 3150 6250 50  0001 C CNN
